Commit message: [easyhec]: Change logging setting.

File: assets/franka/urdf/franka_another.urdf (robot description, URDF)
Before this commit: robot panda, 12 links, 11 joints
Links:
- added link panda_ball, mass 0.1; collision sphere radius=0.01; visual sphere radius=0.01
- link panda_hand: mass None -> 0.1
- link panda_leftfinger: mass None -> 0.1
- link panda_link0: mass None -> 0.1
- link panda_link1: mass None -> 0.1
- link panda_link2: mass None -> 0.1
- link panda_link3: mass None -> 0.1
- link panda_link4: mass None -> 0.1
- link panda_link5: mass None -> 0.1
- link panda_link6: mass None -> 0.1
- link panda_link7: mass None -> 0.1
- link panda_link8: mass None -> 0.1
- link panda_rightfinger: mass None -> 0.1
Joints:
- added joint panda_ball_joint: type fixed, parent panda_hand, child panda_ball, origin xyz=0 0 0.1 rpy=0 0 0
- joint panda_finger_joint1: limit lower=0.0 upper=0.04 effort=20 velocity=0.2 -> lower=0.0 upper=0.00 effort=20 velocity=0.2
- joint panda_finger_joint2: limit lower=0.0 upper=0.04 effort=20 velocity=0.2 -> lower=0.0 upper=0.00 effort=20 velocity=0.2
